File: Robotor 2019/Tribot/Tribot.kicad_pcb (KiCad board)
At the start: 2 copper layers, 223.3 x 130.3 mm, 98 parts, among them J1 Conn_01x03_Male, J2 Conn_01x04_Female, J3 USB_B_Mini, J4 Conn_01x04_Female, J5 Conn_01x04_Female, J7 Conn_01x03_Female, J8 Conn_01x03_Female, M1 Motor_DC, M2 Motor_DC, SW1 SW_Push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

Commit message: Just like 2 damn tracks, nothing important, everything still seems to work.
Routing:
- net Net-(SW_PIN1-Pad1): track 0.00 -> 82.5 mm, vias 0 -> 1
- net Net-(SW_PIN1-Pad2): track 0.00 -> 80.8 mm, vias 0 -> 1
- net EnA_B: track 74.6 -> 82.8 mm
- net OSC-IN: track 78.9 -> 78.3 mm
Changed lines of the file:
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@@
     (thickness 1.6)
     (drawings 141)
-    (tracks 943)
+    (tracks 969)
     (zones 0)
     (modules 98)
@@
   (page A4)
   (layers
-    (0 F.Cu signal)
+    (0 F.Cu signal hide)
     (31 B.Cu signal)
     (32 B.Adhes user)
@@
     (40 Dwgs.User user)
     (41 Cmts.User user)
-    (42 Eco1.User user)
+    (42 Eco1.User user hide)
     (43 Eco2.User user hide)
     (44 Edge.Cuts user)
@@
   (segment (start 108.44 144.78) (end 108.44 142.22) (width 0.39) (layer B.Cu) (net 7))
   (via (at 52.832 138.684) (size 1.2) (drill 0.8) (layers F.Cu B.Cu) (net 7))
-  (segment (start 72.136 138.684) (end 52.832 138.684) (width 0.39) (layer B.Cu) (net 7))
-  (segment (start 102.527372 132.957372) (end 77.862628 132.957372) (width 0.39) (layer B.Cu) (net 7))
   (segment (start 110.49 140.17) (end 109.74 140.17) (width 0.39) (layer B.Cu) (net 7))
-  (segment (start 109.74 140.17) (end 102.527372 132.957372) (width 0.39) (layer B.Cu) (net 7))
-  (segment (start 72.136 138.684) (end 77.862628 132.957372) (width 0.39) (layer B.Cu) (net 7))
+  (segment (start 107.912 140.17) (end 110.49 140.17) (width 0.39) (layer B.Cu) (net 7))
+  (segment (start 102.235 134.493) (end 107.912 140.17) (width 0.39) (layer B.Cu) (net 7))
+  (segment (start 76.327 134.493) (end 102.235 134.493) (width 0.39) (layer B.Cu) (net 7))
+  (segment (start 52.832 138.684) (end 72.136 138.684) (width 0.39) (layer B.Cu) (net 7))
+  (segment (start 72.136 138.684) (end 76.327 134.493) (width 0.39) (layer B.Cu) (net 7))
   (segment (start 55.372 132.4365) (end 55.376 132.4325) (width 0.25) (layer F.Cu) (net 8))
   (segment (start 53.848 137.668) (end 53.848 136.398) (width 0.25) (layer F.Cu) (net 8))
@@
   (segment (start 78.74 130.556) (end 77.978 129.794) (width 0.25) (layer F.Cu) (net 74))
   (segment (start 102.108 130.556) (end 78.74 130.556) (width 0.25) (layer F.Cu) (net 74))
-  (segment (start 113.962 152.701001) (end 115.062 152.701001) (width 0.25) (layer F.Cu) (net 75))
   (segment (start 69.338 128.52) (end 72.644 131.826) (width 0.25) (layer F.Cu) (net 75))
-  (segment (start 72.644 131.826) (end 108.966 131.826) (width 0.25) (layer F.Cu) (net 75))
-  (segment (start 108.966 131.826) (end 112.522 135.382) (width 0.25) (layer F.Cu) (net 75))
-  (segment (start 112.522 135.382) (end 112.522 151.261001) (width 0.25) (layer F.Cu) (net 75))
   (segment (start 59.7885 128.52) (end 69.338 128.52) (width 0.25) (layer F.Cu) (net 75))
-  (segment (start 112.522 151.261001) (end 113.962 152.701001) (width 0.25) (layer F.Cu) (net 75))
+  (segment (start 116.162 152.701001) (end 119.253 149.610001) (width 0.25) (layer F.Cu) (net 75))
+  (segment (start 115.062 152.701001) (end 116.162 152.701001) (width 0.25) (layer F.Cu) (net 75))
+  (segment (start 119.253 149.610001) (end 119.253 133.985) (width 0.25) (layer F.Cu) (net 75))
+  (segment (start 117.094 131.826) (end 108.585 131.826) (width 0.25) (layer F.Cu) (net 75))
+  (segment (start 119.253 133.985) (end 117.094 131.826) (width 0.25) (layer F.Cu) (net 75))
+  (segment (start 72.644 131.826) (end 108.585 131.826) (width 0.25) (layer F.Cu) (net 75))
   (segment (start 106.934 148.082) (end 106.934 147.828) (width 0.25) (layer F.Cu) (net 76))
   (segment (start 105.664 136.144) (end 106.934 137.414) (width 0.25) (layer F.Cu) (net 76))
@@
   (segment (start 69.6 128.02) (end 59.7885 128.02) (width 0.25) (layer F.Cu) (net 80))
   (segment (start 72.771 131.191) (end 69.6 128.02) (width 0.25) (layer F.Cu) (net 80))
-  (segment (start 110.617 131.191) (end 72.771 131.191) (width 0.25) (layer F.Cu) (net 80))
+  (segment (start 123.698 151.554) (end 120.015 147.871) (width 0.25) (layer F.Cu) (net 80))
   (segment (start 123.698 152.654) (end 123.698 151.554) (width 0.25) (layer F.Cu) (net 80))
-  (segment (start 122.512 150.368) (end 115.062 150.368) (width 0.25) (layer F.Cu) (net 80))
-  (segment (start 115.062 150.368) (end 113.284 148.59) (width 0.25) (layer F.Cu) (net 80))
-  (segment (start 113.284 148.59) (end 113.284 133.858) (width 0.25) (layer F.Cu) (net 80))
-  (segment (start 123.698 151.554) (end 122.512 150.368) (width 0.25) (layer F.Cu) (net 80))
-  (segment (start 113.284 133.858) (end 110.617 131.191) (width 0.25) (layer F.Cu) (net 80))
+  (segment (start 120.015 147.871) (end 120.015 133.604) (width 0.25) (layer F.Cu) (net 80))
+  (segment (start 117.602 131.191) (end 110.363 131.191) (width 0.25) (layer F.Cu) (net 80))
+  (segment (start 120.015 133.604) (end 117.602 131.191) (width 0.25) (layer F.Cu) (net 80))
+  (segment (start 110.617 131.191) (end 110.363 131.191) (width 0.25) (layer F.Cu) (net 80))
+  (segment (start 110.363 131.191) (end 72.771 131.191) (width 0.25) (layer F.Cu) (net 80))
   (segment (start 235.712 72.644) (end 240.284 72.644) (width 0.39) (layer B.Cu) (net 81))
   (segment (start 216.916 69.596) (end 216.916 75.438) (width 0.8) (layer B.Cu) (net 81))
@@
   (segment (start 255.27 68.072) (end 254.254 69.088) (width 0.39) (layer B.Cu) (net 83))
   (segment (start 255.27 66.548) (end 255.27 68.072) (width 0.39) (layer B.Cu) (net 83))
+  (segment (start 124.296249 118.781751) (end 116.549249 118.781751) (width 0.25) (layer B.Cu) (net 84))
+  (segment (start 124.968 118.11) (end 124.296249 118.781751) (width 0.25) (layer B.Cu) (net 84))
+  (segment (start 116.549249 118.781751) (end 115.062 120.269) (width 0.25) (layer B.Cu) (net 84))
+  (segment (start 115.062 120.269) (end 115.062 134.62) (width 0.25) (layer B.Cu) (net 84))
+  (segment (start 115.062 134.62) (end 115.062 134.62) (width 0.25) (layer B.Cu) (net 84))
+  (via (at 115.062 134.62) (size 1.2) (drill 0.8) (layers F.Cu B.Cu) (net 84))
+  (segment (start 68.56 129.52) (end 59.7885 129.52) (width 0.25) (layer F.Cu) (net 84))
+  (segment (start 72.136 133.096) (end 68.56 129.52) (width 0.25) (layer F.Cu) (net 84))
+  (segment (start 102.108 133.096) (end 72.136 133.096) (width 0.25) (layer F.Cu) (net 84))
+  (segment (start 115.062 134.62) (end 103.632 134.62) (width 0.25) (layer F.Cu) (net 84))
+  (segment (start 103.632 134.62) (end 102.108 133.096) (width 0.25) (layer F.Cu) (net 84))
+  (segment (start 123.171949 116.313949) (end 116.858051 116.313949) (width 0.25) (layer B.Cu) (net 85))
+  (segment (start 116.858051 116.313949) (end 114.3 118.872) (width 0.25) (layer B.Cu) (net 85))
+  (segment (start 114.3 118.872) (end 114.3 132.715) (width 0.25) (layer B.Cu) (net 85))
+  (segment (start 114.3 132.715) (end 114.3 132.969) (width 0.25) (layer B.Cu) (net 85))
+  (segment (start 114.3 132.969) (end 113.538 133.731) (width 0.25) (layer B.Cu) (net 85))
+  (segment (start 113.538 133.731) (end 105.791 133.731) (width 0.25) (layer B.Cu) (net 85))
+  (segment (start 105.791 133.731) (end 105.283 133.223) (width 0.25) (layer B.Cu) (net 85))
+  (segment (start 105.283 133.223) (end 105.283 133.223) (width 0.25) (layer B.Cu) (net 85))
+  (via (at 105.283 133.223) (size 1.2) (drill 0.8) (layers F.Cu B.Cu) (net 85))
+  (segment (start 68.949 129.02) (end 59.7885 129.02) (width 0.25) (layer F.Cu) (net 85))
+  (segment (start 72.39 132.461) (end 68.949 129.02) (width 0.25) (layer F.Cu) (net 85))
+  (segment (start 105.283 133.223) (end 104.521 132.461) (width 0.25) (layer F.Cu) (net 85))
+  (segment (start 104.521 132.461) (end 72.39 132.461) (width 0.25) (layer F.Cu) (net 85))
   (zone (net 2) (net_name GND) (layer F.Cu) (hatch edge 0.508)
     (connect_pads (clearance 0.508))
