File: Robotor 2019/Line Follower 2/Line Follower 2.sch (KiCad schematic (older format))
At the start: 101 parts, among them J1 Conn_01x03_Male, J2 Conn_01x04_Female, J3 USB_B_Mini, J4 Conn_01x03_Female, J5 Conn_01x03_Female, J7 Conn_01x03_Female, J8 Conn_01x03_Female, M1 Motor_DC, M2 Motor_DC, SW1 SW_Push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

Commit message: no message
Parts:
- removed D10: D, Diode_THT:D_A-405_P5.08mm_Vertical_AnodeUp, symbol Device:D
- removed J1: Conn_01x03_Male, Connector_Wire:SolderWirePad_1x03_P5.715mm_Drill2mm, symbol Connector:Conn_01x03_Male
- removed J3: USB_B_Mini, Connector_USB:USB_Mini-B_Lumberg_2486_01_Horizontal, symbol Connector:USB_B_Mini
- removed R11: 100k, Resistor_SMD:R_0805_2012Metric_Pad1.15x1.40mm_HandSolder, symbol Device:R
- removed U3: AMS1117-5.0, Package_TO_SOT_SMD:SOT-223-3_TabPin2, symbol Regulator_Linear:AMS1117-5.0
- added D11: LED, LED_SMD:LED_0805_2012Metric_Pad1.15x1.40mm_HandSolder, symbol Device:LED
- added J1: Conn_01x02, Connector_PinSocket_2.54mm:PinSocket_1x02_P2.54mm_Vertical, symbol Connector_Generic:Conn_01x02
- added SW2, SW3: SW_Push, Button_Switch_SMD:SW_SPST_CK_RS282G05A3, symbol Switch:SW_Push
- added U3: L78L05_SOT89, Package_TO_SOT_SMD:SOT-89-3_Handsoldering, symbol Regulator_Linear:L78L05_SOT89
- CP5, CP6: footprint Capacitor_SMD:CP_Elec_4x5.3 -> Capacitor_SMD:CP_Elec_10x10
- D1, D2, D3, D4, D5, D6, D7, D8: footprint Diode_THT:D_A-405_P5.08mm_Vertical_AnodeUp -> Diode_SMD:D_1206_3216Metric_Pad1.42x1.75mm_HandSolder
- R10, R9: value 1R -> 10K
- R2: footprint Resistor_SMD:R_0805_2012Metric_Pad1.15x1.40mm_HandSolder -> Resistor_SMD:R_1206_3216Metric_Pad1.42x1.75mm_HandSolder
- R3: value 1K5 -> 500
- SW1: footprint Button_Switch_SMD:SW_Push_1P1T_NO_6x6mm_H9.5mm -> Button_Switch_SMD:SW_SPST_CK_RS282G05A3
- Y1: footprint Crystal:Crystal_SMD_SeikoEpson_MA505-2Pin_12.7x5.1mm -> Crystal:Crystal_SMD_0603-2Pin_6.0x3.5mm_HandSoldering
Connections:
- net labels added: LED1, LED2
- net labels removed: EXT_VCC, PA11, PA12
- wire segments 294 -> 290
Other:
- moved on the sheet: C1, C4, C5, D9, M1, R1, R20, Y1
