File: Robotor 2019/Tribot STM32/Tribot STM32.kicad_pcb (KiCad board)
At the start: 2 copper layers, 223.3 x 130.3 mm, 98 parts, among them J1 Conn_01x03_Male, J2 Conn_01x04_Female, J3 USB_B_Mini, J4 Conn_01x04_Female, J5 Conn_01x04_Female, J7 Conn_01x03_Female, J8 Conn_01x03_Female, M1 Motor_DC, M2 Motor_DC, SW1 SW_Push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

Commit message: no message
Parts:
- SW1, SW2: footprint Button_Switch_SMD:SW_Push_1P1T_NO_6x6mm_H9.5mm -> Button_Switch_SMD:SW_SPST_EVQPE1
- moved C4 2.03 mm to (119.1, 123.2)
- moved Y1 1.14 mm to (120.3, 134.6)
Routing:
- net M1IN1_B: track 136.0 -> 123.6 mm
- net Net-(SW1-Pad2): track 62.6 -> 51.9 mm
- net Net-(SW2-Pad2): track 74.2 -> 67.6 mm
- net M2IN1_B: track 157.8 -> 151.8 mm
- net M1IN2_B: track 139.9 -> 134.3 mm
- net OSC32-IN: track 121.9 -> 127.4 mm
- net M2IN2_B: track 159.4 -> 154.7 mm
- net S3: track 13.7 -> 10.4 mm
- net OSC32-OUT: track 95.8 -> 97.7 mm
- net US1P_IN: track 15.8 -> 16.3 mm
