File: Robotor 2019/Tribot 32u4/Tribot 32u4.kicad_pcb (KiCad board)
At the start: 2 copper layers, 243.9 x 151.5 mm, 89 parts, among them J1 Conn_01x03_Male, J10 Conn_01x04, J11 Conn_01x04, J2 Conn_01x01, J3 USB_B_Mini, J4 Conn_01x04_Female, J5 Conn_01x04_Female, J6 AVR-ISP-6, J7 Conn_01x03_Female, J8 Conn_01x03_Female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

Commit message: Schemele nu au nicio schimbare, doar am miscat putin textul sa se vada bine la imprimanta.
Programul am mai schimbat variabilele si vreau sa vad daca merge bine.
Parts:
- moved J2 23.1 mm to (59.8, 143.5)
- moved R12 23.1 mm to (47.9, 167.4)
- moved R17 23.1 mm to (53.8, 128.5)
- moved R2 23.1 mm to (61.7, 121.0)
- moved U5 23.1 mm to (47.9, 159.8)
- moved U7 23.1 mm to (47.9, 144.8)
- moved C15 23.1 mm to (54.3, 163.6)
- moved R13 23.1 mm to (54.3, 158.0)
- moved REF** 23.1 mm to (115.5, 130.3)
- moved U4 23.1 mm to (47.5, 136.3)
- moved US_PIN4 23.1 mm to (94.8, 153.7)
- moved CP6 23.1 mm to (223.9, 80.7)
- moved D2 23.1 mm to (201.6, 48.2)
- moved D3 23.1 mm to (201.8, 63.2)
- moved D9 23.1 mm to (240.8, 93.4)
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Routing:
- net Net-(D9-Pad1): track 0.00 -> 2.74 mm
Other:
- outline, holes or cut-outs redrawn

Commit message: Honestly I don't even remember
Parts:
- moved J4 7.49 mm to (193.1, 69.6), turned to 180 degrees
Routing:
- net US1_OUT: track 90.3 -> 74.1 mm
- net US1_IN: track 90.8 -> 80.7 mm
- net +5V: track 294.1 -> 296.8 mm
Changed lines of the file:
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@@
     (thickness 1.6)
     (drawings 132)
-    (tracks 602)
+    (tracks 597)
     (zones 0)
     (modules 89)
@@
   )
   (setup
-    (last_trace_width 0.25)
+    (last_trace_width 0.39)
     (user_trace_width 0.39)
     (user_trace_width 0.8)
@@
   )
   (module Connector_PinHeader_2.54mm:PinHeader_1x04_P2.54mm_Vertical (layer F.Cu)
-    (at 193.2559 62.1538)
+    (at 193.08572 69.6468 180)
     (descr "Through hole straight pin header, 1x04, 2.54mm pitch, single row")
     (tags "Through hole pin header THT 1x04 2.54mm single row")
@@
     (fp_line (start 1.27 -1.27) (end 1.27 8.89) (layer F.Fab) (width 0.1))
     (fp_line (start -0.635 -1.27) (end 1.27 -1.27) (layer F.Fab) (width 0.1))
-    (pad 4 thru_hole oval (at 0 7.62) (size 1.7 1.7) (drill 1) (layers *.Cu *.Mask)
+    (pad 4 thru_hole oval (at 0 7.62 180) (size 1.7 1.7) (drill 1) (layers *.Cu *.Mask)
       (net 3 +5V))
-    (pad 3 thru_hole oval (at 0 5.08) (size 1.7 1.7) (drill 1) (layers *.Cu *.Mask)
+    (pad 3 thru_hole oval (at 0 5.08 180) (size 1.7 1.7) (drill 1) (layers *.Cu *.Mask)
       (net 17 US1_IN))
-    (pad 2 thru_hole oval (at 0 2.54) (size 1.7 1.7) (drill 1) (layers *.Cu *.Mask)
+    (pad 2 thru_hole oval (at 0 2.54 180) (size 1.7 1.7) (drill 1) (layers *.Cu *.Mask)
       (net 16 US1_OUT))
-    (pad 1 thru_hole rect (at 0 0) (size 1.7 1.7) (drill 1) (layers *.Cu *.Mask)
+    (pad 1 thru_hole rect (at 0 0 180) (size 1.7 1.7) (drill 1) (layers *.Cu *.Mask)
       (net 2 GND))
     (model ${KISYS3DMOD}/Connector_PinHeader_2.54mm.3dshapes/PinHeader_1x04_P2.54mm_Vertical.wrl
@@
   (segment (start 218.1987 98.1583) (end 221.1324 98.1583) (width 0.39) (layer F.Cu) (net 3))
   (segment (start 213.6775 93.6371) (end 218.1987 98.1583) (width 0.39) (layer F.Cu) (net 3))
-  (segment (start 208.3989 73.2663) (end 209.6389 73.2663) (width 0.39) (layer B.Cu) (net 3))
-  (segment (start 195.546319 73.2663) (end 208.3989 73.2663) (width 0.39) (layer B.Cu) (net 3))
-  (segment (start 193.2559 70.975881) (end 195.546319 73.2663) (width 0.39) (layer B.Cu) (net 3))
-  (segment (start 193.2559 69.7738) (end 193.2559 70.975881) (width 0.39) (layer B.Cu) (net 3))
   (segment (start 262.251678 80.01605) (end 262.251678 56.130678) (width 0.39) (layer F.Cu) (net 3))
   (segment (start 262.251678 56.130678) (end 261.4041 55.2831) (width 0.39) (layer F.Cu) (net 3))
@@
   (segment (start 234.2187 94.4679) (end 240.7793 94.4679) (width 0.39) (layer F.Cu) (net 3))
   (segment (start 229.3493 89.5985) (end 234.2187 94.4679) (width 0.39) (layer F.Cu) (net 3))
+  (segment (start 209.6389 73.2663) (end 206.41818 73.2663) (width 0.39) (layer B.Cu) (net 3))
+  (segment (start 195.17868 62.0268) (end 193.08572 62.0268) (width 0.39) (layer B.Cu) (net 3))
+  (segment (start 206.41818 73.2663) (end 195.17868 62.0268) (width 0.39) (layer B.Cu) (net 3))
   (segment (start 52.0125 160.2837) (end 54.2925 162.5637) (width 0.39) (layer B.Cu) (net 4))
   (segment (start 52.0125 156.9787) (end 52.0125 160.2837) (width 0.39) (layer B.Cu) (net 4))
@@
   (segment (start 251.2949 78.4098) (end 240.1316 78.4098) (width 0.39) (layer B.Cu) (net 16))
   (segment (start 240.1316 78.4098) (end 226.6061 91.9353) (width 0.39) (layer B.Cu) (net 16))
-  (segment (start 226.6061 91.9353) (end 202.5015 91.9353) (width 0.39) (layer B.Cu) (net 16))
-  (segment (start 202.5015 91.9353) (end 189.0649 78.4987) (width 0.39) (layer B.Cu) (net 16))
-  (segment (start 189.0649 78.4987) (end 189.0649 66.5607) (width 0.39) (layer B.Cu) (net 16))
-  (segment (start 190.9318 64.6938) (end 193.2559 64.6938) (width 0.39) (layer B.Cu) (net 16))
-  (segment (start 189.0649 66.5607) (end 190.9318 64.6938) (width 0.39) (layer B.Cu) (net 16))
-  (segment (start 192.053819 67.2338) (end 190.1825 69.105119) (width 0.39) (layer B.Cu) (net 17))
-  (segment (start 193.2559 67.2338) (end 192.053819 67.2338) (width 0.39) (layer B.Cu) (net 17))
-  (segment (start 190.1825 69.105119) (end 190.1825 77.8637) (width 0.39) (layer B.Cu) (net 17))
-  (segment (start 190.1825 77.8637) (end 202.9841 90.6653) (width 0.39) (layer B.Cu) (net 17))
-  (segment (start 202.9841 90.6653) (end 225.2853 90.6653) (width 0.39) (layer B.Cu) (net 17))
+  (segment (start 193.08572 67.1068) (end 194.3862 67.1068) (width 0.39) (layer B.Cu) (net 16))
+  (segment (start 219.2147 91.9353) (end 226.6061 91.9353) (width 0.39) (layer B.Cu) (net 16))
+  (segment (start 194.3862 67.1068) (end 219.2147 91.9353) (width 0.39) (layer B.Cu) (net 16))
   (segment (start 225.2853 90.6653) (end 241.3635 74.5871) (width 0.39) (layer B.Cu) (net 17))
   (segment (start 241.3635 74.5871) (end 251.6251 74.5871) (width 0.39) (layer B.Cu) (net 17))
   (segment (start 253.8349 76.7969) (end 253.8349 78.4098) (width 0.39) (layer B.Cu) (net 17))
   (segment (start 251.6251 74.5871) (end 253.8349 76.7969) (width 0.39) (layer B.Cu) (net 17))
+  (segment (start 220.386301 90.6653) (end 225.2853 90.6653) (width 0.39) (layer B.Cu) (net 17))
+  (segment (start 194.287801 64.5668) (end 220.386301 90.6653) (width 0.39) (layer B.Cu) (net 17))
+  (segment (start 193.08572 64.5668) (end 194.287801 64.5668) (width 0.39) (layer B.Cu) (net 17))
   (segment (start 239.678819 80.9498) (end 244.6909 80.9498) (width 0.39) (layer B.Cu) (net 18))
   (segment (start 223.6724 98.1583) (end 223.6724 96.956219) (width 0.39) (layer B.Cu) (net 18))

Commit message: no message
Routing:
- net GND: vias 0 -> 2
Changed lines of the file:
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@@
     (thickness 1.6)
     (drawings 132)
-    (tracks 597)
+    (tracks 599)
     (zones 0)
     (modules 89)
@@
   )
   (setup
-    (last_trace_width 0.39)
+    (last_trace_width 0.25)
     (user_trace_width 0.39)
     (user_trace_width 0.8)
@@
   (segment (start 56.8833 150.7781) (end 57.6833 150.7781) (width 0.39) (layer F.Cu) (net 2))
   (segment (start 57.9283 150.5331) (end 60.6425 150.5331) (width 0.39) (layer F.Cu) (net 2))
+  (via (at 257.81 77.216) (size 1.2) (drill 0.8) (layers F.Cu B.Cu) (net 2))
+  (via (at 200.66 87.503) (size 1.2) (drill 0.8) (layers F.Cu B.Cu) (net 2))
   (segment (start 232.6259 32.2833) (end 234.9245 29.9847) (width 0.39) (layer F.Cu) (net 3))
   (segment (start 232.6259 33.5233) (end 232.6259 32.2833) (width 0.39) (layer F.Cu) (net 3))
